File: Talon SRX Breakout v2/TALON_SRX v2.0.brd (EAGLE design)
At the start: 25.4 x 39.4 mm, 9 parts, among them J1 TALON_SRX_2X5, X1 HEADER_POS5_70634

Commit message: Made Changes
Parts:
- moved R3 1.90 mm to (23.5, 26.7)
Routing:
- net GND: track 29.3 -> 27.4 mm
- net AIN: track 33.8 -> 34.6 mm
Other:
- board text added: "2018/01/15"
- board text removed: "2018/01/13"
Changed lines of the file:
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@@
 <text x="12.7" y="1.905" size="1.016" layer="25" font="vector" ratio="10" align="bottom-center">Robowranglers</text>
 <text x="12.7" y="0.635" size="0.8128" layer="25" font="vector" ratio="12" align="bottom-center">SRX Breakout v2.0</text>
-<text x="1.905" y="37.7825" size="0.8128" layer="25" font="vector" ratio="12" rot="R90" align="top-right">2018/01/13</text>
+<text x="1.5875" y="38.1" size="0.8128" layer="25" font="vector" ratio="12" rot="R90" align="top-right">2018/01/15</text>
 <text x="12.7" y="21.59" size="5.08" layer="26" rot="SMR270" align="center">Bad?</text>
 </plain>
@@
 <element name="A_IO" library="con-molex-c-grid-sl" package="74099-POS3" value="HEADER_POS3_74099" x="12.7" y="33.02"/>
 <element name="R2" library="SparkFun-Passives" package="1206" value="2K2" x="23.495" y="34.29" rot="R90"/>
-<element name="R3" library="SparkFun-Passives" package="1206" value="4K3" x="23.495" y="28.575" rot="R90"/>
+<element name="R3" library="SparkFun-Passives" package="1206" value="4K3" x="23.495" y="26.67" rot="R90"/>
 </elements>
 <signals>
@@
 <contactref element="R2" pad="1"/>
 <contactref element="R3" pad="2"/>
-<wire x1="13.97" y1="5.3975" x2="13.97" y2="23.495" width="0.4064" layer="16"/>
-<wire x1="13.97" y1="23.495" x2="21.9075" y2="31.4325" width="0.4064" layer="16"/>
-<via x="21.9075" y="31.4325" extent="1-16" drill="0.35"/>
-<wire x1="23.495" y1="32.89" x2="23.495" y2="31.75" width="0.4064" layer="1"/>
-<wire x1="23.495" y1="31.75" x2="23.1775" y2="31.4325" width="0.4064" layer="1"/>
-<wire x1="23.1775" y1="31.4325" x2="21.9075" y2="31.4325" width="0.4064" layer="1"/>
-<wire x1="23.495" y1="29.975" x2="23.495" y2="31.115" width="0.4064" layer="1"/>
-<wire x1="23.495" y1="31.115" x2="23.1775" y2="31.4325" width="0.4064" layer="1"/>
+<wire x1="13.97" y1="5.3975" x2="13.97" y2="22.5425" width="0.4064" layer="16"/>
+<wire x1="13.97" y1="22.5425" x2="21.9075" y2="30.48" width="0.4064" layer="16"/>
+<via x="21.9075" y="30.48" extent="1-16" drill="0.35"/>
+<wire x1="23.495" y1="32.89" x2="23.495" y2="31.4325" width="0.4064" layer="1"/>
+<wire x1="23.495" y1="31.4325" x2="22.5425" y2="30.48" width="0.4064" layer="1"/>
+<wire x1="22.5425" y1="30.48" x2="21.9075" y2="30.48" width="0.4064" layer="1"/>
+<wire x1="23.495" y1="28.07" x2="23.495" y2="29.5275" width="0.4064" layer="1"/>
+<wire x1="23.495" y1="29.5275" x2="22.5425" y2="30.48" width="0.4064" layer="1"/>
 </signal>
 <signal name="QUAD_B">
@@
 <wire x1="10.16" y1="33.02" x2="9.525" y2="32.385" width="0.4064" layer="1"/>
 <via x="9.525" y="32.385" extent="1-16" drill="0.35"/>
-<wire x1="23.495" y1="27.175" x2="23.495" y2="17.78" width="0.4064" layer="1"/>
+<wire x1="23.495" y1="25.27" x2="23.495" y2="17.78" width="0.4064" layer="1"/>
 <wire x1="23.495" y1="17.78" x2="22.4155" y2="16.7005" width="0.4064" layer="1"/>
 <wire x1="22.4155" y1="16.7005" x2="22.4155" y2="15.24" width="0.4064" layer="1"/>
@@
 <signal name="N$8">
 <polygon width="0.1524" layer="1" pour="cutout">
-<vertex x="0" y="27.305"/>
-<vertex x="1.905" y="27.305"/>
+<vertex x="0" y="28.2575"/>
+<vertex x="1.905" y="28.2575"/>
 <vertex x="1.905" y="18.415"/>
 <vertex x="3.175" y="17.145"/>
@@
 <vertex x="26.3525" y="40.64"/>
 <vertex x="22.225" y="40.64"/>
-<vertex x="22.5425" y="20.32"/>
-<vertex x="20.6375" y="18.415"/>
-<vertex x="20.6375" y="15.5575"/>
-<vertex x="26.3525" y="15.5575"/>
-</polygon>
-</signal>
+<vertex x="22.225" y="20.0025"/>
+<vertex x="20.0025" y="17.78"/>
+<vertex x="20.0025" y="4.1275"/>
+<vertex x="26.3525" y="4.1275"/>
+</polygon>
+</signal>
